File: PCBs/Base/BeanPad.kicad_sch (KiCad schematic)
At the start: 9 parts, among them J1 Male_Pogo_Connector_01x05, J2 Display, J3 Male_Pogo_Connector_01x05, J5 Male_Pogo_Connector_01x05, SW1 SW_Push, SW2 SW_Push, SW3 SW_Push, U1 XIAO-RP2040-DIP

Commit message: Modules
Parts:
- removed D1: SK6812MINI, LED_SMD:LED_SK6812MINI_PLCC4_3.5x3.5mm_P1.75mm, symbol LED:SK6812MINI
- J1, J3, J5: footprint Conn_Pogo:male_only_connector_5pin_Version3 -> Connector_PinHeader_2.54mm:PinHeader_1x05_P2.54mm_Vertical
Connections:
- net GPIO26: now also SW3.2; no longer SW1.2
- net GPIO28: now also SW1.2; no longer SW3.2
- net INT: now also J1.3 (AUX), J3.3 (AUX), J5.3 (AUX); no longer J1.5 (AUX), J3.5 (AUX), J5.5 (AUX)
- net SCL: now also J1.5 (CLK), J3.5 (CLK), J5.5 (CLK); no longer J1.4 (CLK), J3.4 (CLK), J5.4 (CLK)
- net SDA: now also J1.4 (DATA), J3.4 (DATA), J5.4 (DATA); no longer J1.3 (DATA), J3.3 (DATA), J5.3 (DATA)
- no-connect marks 5 -> 4
Changed lines of the file:
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@@
-	)
-	(no_connect
-		(at 146.05 41.91)
 	)
 	(no_connect
@@
 		)
 	)
-	(label "GPIO4"
-		(at 130.81 41.91 180)
-		(effects
-			(font
-				(size 1.27 1.27)
-			)
-			(justify right bottom)
-		)
-	)
 	(label "INT"
-		(at 257.81 107.95 0)
+		(at 257.81 102.87 0)
 		(effects
 			(font
@@
 	)
 	(label "INT"
-		(at 257.81 135.89 0)
+		(at 257.81 130.81 0)
 		(effects
 			(font
@@
 	)
 	(label "GPIO28"
-		(at 52.07 106.68 0)
+		(at 52.07 80.01 0)
 		(effects
 			(font
@@
 	)
 	(label "SDA"
-		(at 247.65 130.81 180)
+		(at 247.65 133.35 180)
 		(effects
 			(font
@@
 	)
 	(label "SDA"
-		(at 247.65 102.87 180)
+		(at 247.65 105.41 180)
 		(effects
 			(font
@@
 	)
 	(label "GPIO26"
-		(at 52.07 80.01 0)
+		(at 52.07 106.68 0)
 		(effects
 			(font
@@
 	)
 	(label "SCL"
-		(at 247.65 68.58 180)
+		(at 247.65 71.12 180)
 		(effects
 			(font
@@
 	)
 	(label "SCL"
-		(at 247.65 133.35 180)
+		(at 247.65 135.89 180)
 		(effects
 			(font
@@
 	)
 	(label "SDA"
-		(at 247.65 66.04 180)
+		(at 247.65 68.58 180)
 		(effects
 			(font
@@
 	)
 	(label "SCL"
-		(at 247.65 105.41 180)
+		(at 247.65 107.95 180)
 		(effects
 			(font
@@
 	)
 	(label "INT"
-		(at 257.81 71.12 0)
+		(at 257.81 66.04 0)
 		(effects
 			(font
@@
 			)
 		)
-		(property "Footprint" "Conn_Pogo:male_only_connector_5pin_Version3"
+		(property "Footprint" "Connector_PinHeader_2.54mm:PinHeader_1x05_P2.54mm_Vertical"
 			(at 252.73 76.2 0)
 			(effects
@@
 			)
 		)
-		(property "Footprint" "Conn_Pogo:male_only_connector_5pin_Version3"
+		(property "Footprint" "Connector_PinHeader_2.54mm:PinHeader_1x05_P2.54mm_Vertical"
 			(at 252.73 113.03 0)
 			(effects
@@
 	)
 	(symbol
-		(lib_id "power:GND")
-		(at 138.43 49.53 0)
-		(unit 1)
-		(exclude_from_sim no)
-		(in_bom yes)
-		(on_board yes)
-		(dnp no)
-		(fields_autoplaced yes)
-		(property "Reference" "#PWR010"
-			(at 138.43 55.88 0)
-			(effects
-				(font
-					(size 1.27 1.27)
-				)
-				(hide yes)
-			)
-		)
-		(property "Value" "GND"
-			(at 138.43 54.61 0)
-			(effects
-				(font
-					(size 1.27 1.27)
-				)
-			)
-		)
-		(property "Footprint" ""
-			(at 138.43 49.53 0)
-			(effects
-				(font
-					(size 1.27 1.27)
-				)
-				(hide yes)
-			)
-		)
-		(property "Datasheet" ""
-			(at 138.43 49.53 0)
-			(effects
-				(font
-					(size 1.27 1.27)
-				)
-				(hide yes)
-			)
-		)
-		(property "Description" "Power symbol creates a global label with name \"GND\" , ground"
-			(at 138.43 49.53 0)
-			(effects
-				(font
-					(size 1.27 1.27)
-				)
-				(hide yes)
-			)
-		)
-		(pin "1"
-		)
-		(instances
-			(project ""
-				(path "/0fada3d2-b91b-45d1-ab99-8eb3053f21b6"
-					(reference "#PWR010")
-					(unit 1)
-				)
-			)
-		)
-	)
-	(symbol
 		(lib_id "power:+3V3")
 		(at 165.1 87.63 270)
@@
 	)
 	(symbol
-		(lib_id "LED:SK6812MINI")
-		(at 138.43 41.91 0)
-		(unit 1)
-		(exclude_from_sim no)
-		(in_bom yes)
-		(on_board yes)
-		(dnp no)
-		(fields_autoplaced yes)
-		(property "Reference" "D1"
-			(at 151.13 35.4898 0)
-			(effects
-				(font
-					(size 1.27 1.27)
-				)
-			)
-		)
-		(property "Value" "SK6812MINI"
-			(at 151.13 38.0298 0)
-			(effects
-				(font
-					(size 1.27 1.27)
-				)
-			)
-		)
-		(property "Footprint" "LED_SMD:LED_SK6812MINI_PLCC4_3.5x3.5mm_P1.75mm"
-			(at 139.7 49.53 0)
-			(effects
-				(font
-					(size 1.27 1.27)
-				)
-				(justify left top)
-				(hide yes)
-			)
-		)
-		(property "Datasheet" "https://cdn-shop.adafruit.com/product-files/2686/SK6812MINI_REV.01-1-2.pdf"
-			(at 140.97 51.435 0)
-			(effects
-				(font
-					(size 1.27 1.27)
-				)
-				(justify left top)
-				(hide yes)
-			)
-		)
-		(property "Description" "RGB LED with integrated controller"
-			(at 138.43 41.91 0)
-			(effects
-				(font
-					(size 1.27 1.27)
-				)
-				(hide yes)
-			)
-		)
-		(pin "2"
-		)
-		(pin "3"
-		)
-		(pin "1"
-		)
-		(pin "4"
-		)
-		(instances
-			(project ""
-				(path "/0fada3d2-b91b-45d1-ab99-8eb3053f21b6"
-					(reference "D1")
-					(unit 1)
-				)
-			)
-		)
-	)
-	(symbol
 		(lib_id "power:VCC")
 		(at 247.65 60.96 90)
@@
 			)
 		)
-		(property "Footprint" "Conn_Pogo:male_only_connector_5pin_Version3"
+		(property "Footprint" "Connector_PinHeader_2.54mm:PinHeader_1x05_P2.54mm_Vertical"
 			(at 252.73 140.97 0)
 			(effects
@@
 					(unit 1)
 				)
-			)
-		)
-	)
-	(symbol
-		(lib_id "power:VCC")
-		(at 138.43 34.29 0)
-		(unit 1)
-		(exclude_from_sim no)
-		(in_bom yes)
-		(on_board yes)
-		(dnp no)
-		(fields_autoplaced yes)
-		(property "Reference" "#PWR09"
-			(at 138.43 38.1 0)
-			(effects
-				(font
-					(size 1.27 1.27)
-				)
-				(hide yes)
-			)
-		)
-		(property "Value" "VCC"
-			(at 138.43 29.21 0)
-			(effects
-				(font
-					(size 1.27 1.27)
-				)
-			)
-		)
-		(property "Footprint" ""
-			(at 138.43 34.29 0)
-			(effects
-				(font
-					(size 1.27 1.27)
-				)
-				(hide yes)
-			)
-		)
-		(property "Datasheet" ""
-			(at 138.43 34.29 0)
-			(effects
-				(font
-					(size 1.27 1.27)
-				)
-				(hide yes)
-			)
-		)
-		(property "Description" "Power symbol creates a global label with name \"VCC\""
-			(at 138.43 34.29 0)
-			(effects
-				(font
-					(size 1.27 1.27)
-				)
-				(hide yes)
-			)
-		)
-		(pin "1"
-		)
-		(instances
-			(project ""
-				(path "/0fada3d2-b91b-45d1-ab99-8eb3053f21b6"
-					(reference "#PWR09")
-					(unit 1)
-				)
