File: PCBs/Base/BeanPad.kicad_pcb (KiCad board)
At the start: 2 copper layers, 80 x 80 mm, 10 parts, among them J1 Male_Pogo_Connector_01x05, J2 Display, J3 Male_Pogo_Connector_01x05, J5 Male_Pogo_Connector_01x05, SW1 SW_Push, SW2 SW_Push, SW3 SW_Push, U1 XIAO-RP2040-DIP

Commit message: Fix PCB and Pictures
Parts:
- added G***: LOGO, LOGO, F.Cu at (129.6, 133.7)
- added G***: LOGO, LOGO, B.Cu at (118.0, 131.0)
Other:
- outline, holes or cut-outs redrawn
