File: PCBs/Macro/Macro.kicad_pcb (KiCad board)
At the start: 2 copper layers, 80 x 51 mm, 11 parts, among them J1 Male_Pogo_Connector_01x05, J2 Male_Pogo_Connector_01x05, J3 Male_Pogo_Connector_01x05, J4 Male_Pogo_Connector_01x05, SW1 SW_Push, SW2 SW_Push, SW3 SW_Push, SW4 SW_Push, U1 XIAO-RP2040-DIP

Commit message: Fix PCB and Pictures
Parts:
- added G***: LOGO, LOGO, F.Cu at (162.0, 110.0)
- added G***: LOGO, LOGO, B.Cu at (125.0, 107.0)
Other:
- outline, holes or cut-outs redrawn
