File: PCBs/Knobs/Knobs.kicad_pcb (KiCad board)
At the start: 2 copper layers, 80 x 40 mm, 15 parts, among them J1 Male_Pogo_Connector_01x05, J2 Male_Pogo_Connector_01x05, J3 Male_Pogo_Connector_01x05, J4 Male_Pogo_Connector_01x05, SW1 RotaryEncoder_Switch, SW2 RotaryEncoder_Switch, U1 XIAO-RP2040-DIP

Commit message: Finished Designing
Parts:
- removed R1, R2, R3, R4, R5, R6: 10k, Resistor_THT:R_Axial_DIN0207_L6.3mm_D2.5mm_P10.16mm_Horizontal
- removed REF** (x2): MountingHole_3.2mm_M3, MountingHole:MountingHole_3.2mm_M3
Routing:
- net +3V3: track 86.2 -> 0.00 mm
- net /GPIO27: track 48.2 -> 46.5 mm

Commit message: Fix PCB and Pictures
Parts:
- added G***: LOGO, LOGO, B.Cu at (166.0, 65.0)
- added REF**: MountingHole_3.2mm_M3, MountingHole:MountingHole_3.2mm_M3, F.Cu at (174.6, 80.6)
- added REF**: MountingHole_3.2mm_M3, MountingHole:MountingHole_3.2mm_M3, F.Cu at (105.4, 80.6)
Other:
- outline, holes or cut-outs redrawn
